File: BlinkIR.sch (KiCad schematic (older format))
At the start: 18 parts, among them Q1 Q_Photo_NPN, Q2 Q_Photo_NPN, Q3 Q_Photo_NPN, U1 ATtiny10-TS

Commit message: software retargeted to ATTiny10 and dropped uart Schmatic work finished rev1
Parts:
- removed BT1: Battery_Cell, Battery_Holders:Keystone_3034_1x20mm-CoinCell, symbol Device:Battery_Cell
- added J1, J2, J3: Conn_01x01, Mounting_Holes:MountingHole_4.3mm_M4_ISO7380_Pad, symbol Connector_Generic:Conn_01x01
- D2, D3, D4: footprint (none) -> LEDs:LED_0805
- Q1, Q2, Q3: footprint (none) -> LEDs:LED_D3.0mm_Horizontal_O1.27mm_Z2.0mm
Connections:
- wire segments 55 -> 59
Other:
- moved on the sheet: U1
